File: hw/circle.kicad_pcb (KiCad board)
At the start: 4 copper layers, 46 x 46 mm, 50 parts, among them J1 CONN_01X02, J2 USB_OTG, J3 CONN_01X03, J4 CONN_02X05, J5 CONN_01X03, J6 CONN_01X06, U1 STM32F303CCTx, U2 AS5048A, U3 DRV8312, U4 INA240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

Commit message: rev.A sent to fab
Parts:
- added D1: LED_Small, LEDs:LED_0603, F.Cu at (85.2, 88.2)
- added R7: 0R05, Resistors_SMD:R_0603, F.Cu at (82.5, 92.8)
- R2: footprint Resistors_SMD:R_0805 -> Resistors_SMD:R_0603
- moved C15 4.56 mm to (104.8, 100.5), turned to 90 degrees
- moved C2 2.85 mm to (115.8, 95.8), turned to 315 degrees
- moved C5 1.95 mm to (114.8, 115.5), turned to 45 degrees
- moved C19 1.00 mm to (96.0, 99.0)
- moved R2 0.71 mm to (110.0, 114.5), turned to 0 degrees
- moved C1 0.64 mm to (110.0, 112.5), turned to 180 degrees
- moved R1 0.56 mm to (112.2, 113.0)
- moved C22 0.50 mm to (97.0, 94.5)
- moved C11 0.25 mm to (111.2, 98.5)
- moved C18 0.25 mm to (83.8, 95.5)
- moved C3 0.25 mm to (110.8, 96.0)
- turned C25 to 180 degrees
Connections:
- U1 pad 2: /FAULT -> /RSTB
- U1 pad 27: Net-(U1-Pad27) -> /LED
- U1 pad 39: /RSTA -> /OTW
- U1 pad 40: /RSTB -> /RSTA
- U1 pad 41: /RSTC -> /FAULT
- U1 pad 43: /OTW -> /RSTC
Routing:
- net GND: track 38.8 -> 120.2 mm, vias 19 -> 59
- net +12V: track 15.0 -> 73.9 mm, vias 3 -> 15
- net /OTW: track 0.00 -> 47.4 mm, vias 0 -> 2
- net /RSTA: track 0.00 -> 43.1 mm, vias 0 -> 2
- net /FAULT: track 0.00 -> 42.3 mm, vias 0 -> 2
- net /RSTB: track 0.00 -> 37.0 mm, vias 0 -> 2
- net /RSTC: track 0.00 -> 33.9 mm, vias 0 -> 2
- net /SENSEA: track 2.23 -> 21.6 mm
- net /SENSEB: track 2.23 -> 18.1 mm
- net /VREG: track 0.00 -> 13.8 mm, vias 0 -> 2
- net /AGND: track 0.00 -> 11.0 mm
- net /OSC_IN: track 0.00 -> 8.75 mm
- net +3V3: track 17.4 -> 26.1 mm, vias 6 -> 9
- net /LED: track 0.00 -> 7.54 mm
- net /OSC_OUT: track 0.00 -> 7.42 mm
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- added copper zone on F.Cu, net /AGND
- added copper zone on F.Cu, net /SENSEB
- added copper zone on B.Cu, net GND
- added copper zone on F.Cu, net GND
Other:
- board size 46 x 46 mm -> 46.1 x 45.5 mm
- board text added: "+12V"
- board text added: "12V"
- board text added: "3V3"
- board text added: "4/2017"
- board text added: "A"
- board text added: "B"
- board text added: "G"
- board text added: "GND"
- board text added: "OUTA"
- board text added: "OUTB"
- board text added: "OUTC"
- board text added: "REV. A"
- board text added: "RX"
- board text added: "SLOW-BLDC"
- board text added: "TX"
